Commit message: broke out battery_block into seperate file

File: earth_rover_description/urdf/base/base.urdf.xacro (robot description, xacro)
@@ -1,9 +1,9 @@
 <?xml version="1.0" encoding="UTF-8"?>
 <robot xmlns:xacro="http://www.ros.org/wiki/xacro">
-	<xacro:property name="base_x" value=".2148" />
-	<xacro:property name="base_y" value=".106" />
-	<xacro:property name="base_z" value=".142" />
-	<xacro:property name="shoulder_x" value=".109" />
-	<xacro:property name="shoulder_y" value=".26" />
+	<xacro:property name="base_x" value="0.2148" />
+	<xacro:property name="base_y" value="0.106" />
+	<xacro:property name="base_z" value="0.142" />
+	<xacro:property name="shoulder_x" value="0.109" />
+	<xacro:property name="shoulder_y" value="0.26" />
 	<xacro:property name="hinge_offset" value=".029" />
 	<xacro:macro name="base_block" params="name parent reflect colour">

File: earth_rover_description/urdf/earth_rover.urdf.xacro (robot description, xacro)
@@ -2,6 +2,8 @@
 <robot name="earth_rover" xmlns:xacro="http://www.ros.org/wiki/xacro">
 	<xacro:property name="M_PI" value="3.1415926535897931" />
-	<xacro:include filename="base.urdf.xacro" />
-	<xacro:include filename="wheels.urdf.xacro" />
+	<xacro:property name="fix_base" value="false" />
+	<xacro:include filename="base/base.urdf.xacro" />
+	<xacro:include filename="base/battery_block.urdf.xacro" />
+	<xacro:include filename="wheels/wheels.urdf.xacro" />
 	<xacro:include filename="earth_rover.gazebo.xacro" />
 	<material name="yellow">
@@ -39,25 +41,3 @@
 	<xacro:wheel name="back_left" parent="back_base_link" reflect="1" reflect_y="-1" />
 	<xacro:wheel name="back_right" parent="back_base_link" reflect="-1" reflect_y="-1" />
-	<!-- battery block -->
-	<link name="battery_block_link">
-		<inertial>
-			<!-- from Solid Edge "Battery Block V2 - 22Ah - 24V.asm" -->
-			<origin xyz="-0.09568 0 0.00658" />
-			<mass value="2.401" />
-			<inertia ixx="0.002" iyy="-0.001" izz="-0.001" ixy="0" ixz="0" iyz="0" />
-		</inertial>
-		<visual>
-			<geometry>
-				<mesh filename="package://earth_rover_description/meshes/battery_block.dae" />
-			</geometry>
-		</visual>
-	</link>
-	<gazebo reference="battery_block_link">
-		<selfCollide>false</selfCollide>
-	</gazebo>
-	<joint name="battery_block_joint" type="fixed">
-		<parent link="front_base_link" />
-		<child link="battery_block_link" />
-		<origin xyz="${base_x/2} 0 0" />
-	</joint>
 </robot>

Commit message: broke out xacro properties into properties files for convenience

File: earth_rover_description/urdf/base/base.urdf.xacro (robot description, xacro)
@@ -1,10 +1,5 @@
 <?xml version="1.0" encoding="UTF-8"?>
 <robot xmlns:xacro="http://www.ros.org/wiki/xacro">
-	<xacro:property name="base_x" value="0.2148" />
-	<xacro:property name="base_y" value="0.106" />
-	<xacro:property name="base_z" value="0.142" />
-	<xacro:property name="shoulder_x" value="0.109" />
-	<xacro:property name="shoulder_y" value="0.26" />
-	<xacro:property name="hinge_offset" value=".029" />
+	<xacro:include filename="00-base_properties.xacro" />
 	<xacro:macro name="base_block" params="name parent reflect colour">
 		<link name="${name}_link">

File: earth_rover_description/urdf/earth_rover.urdf.xacro (robot description, xacro)
@@ -6,4 +6,5 @@
 	<xacro:include filename="base/battery_block.urdf.xacro" />
 	<xacro:include filename="wheels/wheels.urdf.xacro" />
+	<!-- <xacro:include filename="ankles/ankles.urdf.xacro" /> -->
 	<xacro:include filename="earth_rover.gazebo.xacro" />
 	<material name="yellow">
@@ -20,5 +21,5 @@
 	</material>
 	<!-- link of convenience, makes things more symmetrical -->
-	<link name="base_link"/>
+	<link name="base_link" />
 	<!-- gazebo doesn't recognise links without mass, but KDL doesn't
 	     like the base link to have inertia, so we have this silly

File: earth_rover_description/urdf/wheels/wheels.urdf.xacro (robot description, xacro)
@@ -1,18 +1,5 @@
 <?xml version="1.0" encoding="UTF-8"?>
 <robot xmlns:xacro="http://www.ros.org/wiki/xacro">
-	<xacro:property name="angle_limit_cw" value="${M_PI/4}" />
-	<xacro:property name="angle_limit_ccw" value="${M_PI/4}" />
-	<xacro:property name="ankle_offset_x" value="0.0914" />
-	<xacro:property name="ankle_offset_y" value="0.140" />
-	<xacro:property name="ankle_offset_z" value="0.051" />
-	<xacro:property name="wheel_offset_y" value=".027" />
-	<xacro:property name="wheel_offset_z" value=".021" />
-	<xacro:property name="wheel_radius" value=".12" />
-	<xacro:property name="wheel_inner_radius" value=".045" />
-	<xacro:property name="wheel_length" value=".09" />
-	<xacro:property name="wheel_mass" value="1.24" />
-	<!-- from standard equation for thick-walled cylinder -->
-	<xacro:property name="wheel_Ixx_Iyy" value="${wheel_mass*(3*(wheel_radius**2 + wheel_inner_radius**2) + wheel_length**2)/12}" />
-	<xacro:property name="wheel_Izz" value="${wheel_mass*(wheel_radius**2 + wheel_inner_radius**2)/2}" />
+	<xacro:include filename="00-wheels_properties.xacro" />
 	<xacro:macro name="wheel" params="name parent reflect reflect_y">
 		<link name="${name}_ankle">
