Commit message: refactoring of wheels urdf model

File: earth_rover_description/urdf/wheels/wheels.urdf.xacro (robot description, xacro)
@@ -53,4 +53,5 @@
 			<material>Gazebo/DarkGrey</material>
 		</gazebo>
+		<!-- Ankle Transmission & Joints -->
 		<joint name="${name}_ankle_joint" type="revolute">
 			<parent link="${parent}" />
@@ -60,11 +61,4 @@
 			<limit lower="-${angle_limit_ccw}" upper="${angle_limit_cw}" effort="7" velocity="15" /> <!-- guesses -->
 		</joint>
-		<joint name="${name}_wheel_joint" type="continuous">
-			<parent link="${name}_ankle" />
-			<child link="${name}_wheel" />
-			<axis xyz="0 1 0" />
-			<origin xyz="0 ${reflect*wheel_offset_y} ${wheel_offset_z}" />
-		</joint>
-		<!-- transmissions needed for gazebo -->
 		<transmission name="${name}_ankle_transmission">
 			<type>transmission_interface/SimpleTransmission</type>
@@ -74,4 +68,5 @@
 			</joint>
 		</transmission>
+		<!-- Wheel Transmition & Joints -->
 		<transmission name="${name}_wheel_transmission">
 			<type>transmission_interface/SimpleTransmission</type>
@@ -81,4 +76,10 @@
 			</joint>
 		</transmission>
+		<joint name="${name}_wheel_joint" type="continuous">
+			<parent link="${name}_ankle" />
+			<child link="${name}_wheel" />
+			<axis xyz="0 1 0" />
+			<origin xyz="0 ${reflect*wheel_offset_y} ${wheel_offset_z}" />
+		</joint>
 	</xacro:macro>
 </robot>
