Commit message: minor refactorings

File: earth_rover_description/urdf/ankles/ankles.urdf.xacro (robot description, xacro)
@@ -1,7 +1,45 @@
 <?xml version="1.0" encoding="UTF-8"?>
 <robot xmlns:xacro="http://www.ros.org/wiki/xacro">
-	<xacro:property name="angle_limit_cw" value="${M_PI/4}" />
-	<xacro:property name="angle_limit_ccw" value="${M_PI/4}" />
-	<xacro:property name="ankle_offset_x" value="0.0914" />
-	<xacro:property name="ankle_offset_y" value="0.140" />
-	<xacro:property name="ankle_offset_z" value="0.051" />
+    <xacro:include filename="00-ankles_properties.xacro" />
+    <xacro:macro name="ankle" params="name parent reflect reflect_y">
+		<link name="${name}_ankle">
+			<inertial>
+				<!-- from Solid Edge "Steering Block.asm" -->
+				<origin xyz="0 ${reflect*(-wheel_offset_y + 0.02493)} ${wheel_offset_z + 0.05588}" />
+				<mass value="0.271" />
+				<inertia ixx="0.01" iyy="0.01" izz="0.01" ixy="0" ixz="0" iyz="0" />
+			</inertial>
+			<visual>
+				<origin xyz="0 ${reflect*wheel_offset_y} ${wheel_offset_z}" rpy="0 0 ${M_PI if reflect == -1 else 0}"/>
+				<geometry>
+					<mesh filename="package://earth_rover_description/meshes/steering_block.dae" />
+				</geometry>
+				<material name="silver"/>
+			</visual>
+			<collision>
+				<origin xyz="0 0 ${ankle_offset_z}" />
+				<geometry>
+					<cylinder radius="0.016" length=".18"/>
+				</geometry>
+			</collision>
+		</link>
+		<gazebo reference="${name}_ankle">
+			<selfCollide>false</selfCollide>
+		</gazebo>
+		<!-- Ankle Transmission & Joints -->
+		<joint name="${name}_ankle_joint" type="revolute">
+			<parent link="${parent}" />
+			<child link="${name}_ankle" />
+			<axis xyz="0 0 1" />
+			<origin xyz="${reflect_y*ankle_offset_x} ${reflect*ankle_offset_y} -${ankle_offset_z}" />
+			<limit lower="-${angle_limit_ccw}" upper="${angle_limit_cw}" effort="7" velocity="15" /> <!-- guesses -->
+		</joint>
+		<transmission name="${name}_ankle_transmission">
+			<type>transmission_interface/SimpleTransmission</type>
+			<actuator name="${name}_ankle_motor" />
+			<joint name="${name}_ankle_joint">
+				<hardwareInterface>hardware_interface/EffortJointInterface</hardwareInterface>
+			</joint>
+		</transmission>
+    </xacro:macro>
+</robot>

File: earth_rover_description/urdf/earth_rover.urdf.xacro (robot description, xacro)
@@ -3,21 +3,10 @@
 	<xacro:property name="M_PI" value="3.1415926535897931" />
 	<xacro:property name="fix_base" value="false" />
+	<xacro:include filename="00-earth_rover_properties.xacro" />
 	<xacro:include filename="base/base.urdf.xacro" />
 	<xacro:include filename="base/battery_block.urdf.xacro" />
 	<xacro:include filename="wheels/wheels.urdf.xacro" />
-	<!-- <xacro:include filename="ankles/ankles.urdf.xacro" /> -->
+	<xacro:include filename="ankles/ankles.urdf.xacro" />
 	<xacro:include filename="earth_rover.gazebo.xacro" />
-	<material name="yellow">
-		<color rgba=".8 .8 0 1" />
-	</material>
-	<material name="black">
-		<color rgba="0 0 0 1" />
-	</material>
-	<material name="green">
-		<color rgba="0 0.8 0 1" />
-	</material>
-	<material name="silver">
-		<color rgba=".8 .8 .8 1" />
-	</material>
 	<!-- link of convenience, makes things more symmetrical -->
 	<link name="base_link" />
@@ -42,3 +31,7 @@
 	<xacro:wheel name="back_left" parent="back_base_link" reflect="1" reflect_y="-1" />
 	<xacro:wheel name="back_right" parent="back_base_link" reflect="-1" reflect_y="-1" />
+	<xacro:ankle name="front_left" parent="front_base_link" reflect="1" reflect_y="1" />
+	<xacro:ankle name="front_right" parent="front_base_link" reflect="-1" reflect_y="1" />
+	<xacro:ankle name="back_left" parent="back_base_link" reflect="1" reflect_y="-1" />
+	<xacro:ankle name="back_right" parent="back_base_link" reflect="-1" reflect_y="-1" />
 </robot>

File: earth_rover_description/urdf/wheels/wheels.urdf.xacro (robot description, xacro)
@@ -3,28 +3,4 @@
 	<xacro:include filename="00-wheels_properties.xacro" />
 	<xacro:macro name="wheel" params="name parent reflect reflect_y">
-		<link name="${name}_ankle">
-			<inertial>
-				<!-- from Solid Edge "Steering Block.asm" -->
-				<origin xyz="0 ${reflect*(-wheel_offset_y + 0.02493)} ${wheel_offset_z + 0.05588}" />
-				<mass value="0.271" />
-				<inertia ixx="0.01" iyy="0.01" izz="0.01" ixy="0" ixz="0" iyz="0" />
-			</inertial>
-			<visual>
-				<origin xyz="0 ${reflect*wheel_offset_y} ${wheel_offset_z}" rpy="0 0 ${M_PI if reflect == -1 else 0}"/>
-				<geometry>
-					<mesh filename="package://earth_rover_description/meshes/steering_block.dae" />
-				</geometry>
-				<material name="silver"/>
-			</visual>
-			<collision>
-				<origin xyz="0 0 ${ankle_offset_z}" />
-				<geometry>
-					<cylinder radius="0.016" length=".18"/>
-				</geometry>
-			</collision>
-		</link>
-		<gazebo reference="${name}_ankle">
-			<selfCollide>false</selfCollide>
-		</gazebo>
 		<link name="${name}_wheel">
 			<inertial>
@@ -53,19 +29,4 @@
 			<material>Gazebo/DarkGrey</material>
 		</gazebo>
-		<!-- Ankle Transmission & Joints -->
-		<joint name="${name}_ankle_joint" type="revolute">
-			<parent link="${parent}" />
-			<child link="${name}_ankle" />
-			<axis xyz="0 0 1" />
-			<origin xyz="${reflect_y*ankle_offset_x} ${reflect*ankle_offset_y} -${ankle_offset_z}" />
-			<limit lower="-${angle_limit_ccw}" upper="${angle_limit_cw}" effort="7" velocity="15" /> <!-- guesses -->
-		</joint>
-		<transmission name="${name}_ankle_transmission">
-			<type>transmission_interface/SimpleTransmission</type>
-			<actuator name="${name}_ankle_motor" />
-			<joint name="${name}_ankle_joint">
-				<hardwareInterface>hardware_interface/EffortJointInterface</hardwareInterface>
-			</joint>
-		</transmission>
 		<!-- Wheel Transmition & Joints -->
 		<transmission name="${name}_wheel_transmission">

Commit message: Model has been restructured; - properties split out - ankles split out - ros_control now initiates with urdf model
Gazebo simulation is functional

File: earth_rover_description/urdf/ankles/ankles.urdf.xacro (robot description, xacro)
@@ -39,5 +39,5 @@
 			<actuator name="${name}_ankle_motor" />
 			<joint name="${name}_ankle_joint">
-				<hardwareInterface>hardware_interface/EffortJointInterface</hardwareInterface>
+				<hardwareInterface>hardware_interface/VelocityJointInterface</hardwareInterface>
 			</joint>
 		</transmission>

File: earth_rover_description/urdf/earth_rover.gazebo.xacro (robot description, xacro)
@@ -1,9 +1,7 @@
 <?xml version="1.0" encoding="UTF-8"?>
 <robot name="earth_rover" xmlns:xacro="http://www.ros.org/wiki/xacro">
-    <xacro:macro name="earth_rover_tags">
+    <xacro:macro name="earth_rover_gazebo_tags">
         <gazebo>
-            <plugin name="gazebo_ros_control" filename="libgazebo_ros_control.so">
-                <robotNamespace>/earth_rover</robotNamespace>
-            </plugin>
+            <plugin name="gazebo_ros_control" filename="libgazebo_ros_control.so" />
         </gazebo>
         <!-- Might need to add stuff here?.... -->

File: earth_rover_description/urdf/earth_rover.urdf.xacro (robot description, xacro)
@@ -9,5 +9,4 @@
 	<xacro:include filename="ankles/ankles.urdf.xacro" />
 	<xacro:include filename="earth_rover.gazebo.xacro" />
-	<!-- link of convenience, makes things more symmetrical -->
 	<link name="base_link" />
 	<!-- gazebo doesn't recognise links without mass, but KDL doesn't
@@ -35,3 +34,4 @@
 	<xacro:ankle name="back_left" parent="back_base_link" reflect="1" reflect_y="-1" />
 	<xacro:ankle name="back_right" parent="back_base_link" reflect="-1" reflect_y="-1" />
+	<xacro:earth_rover_gazebo_tags />
 </robot>
